File: vccs/power.kicad_sch (KiCad schematic)
At the start: 10 parts, among them U3 LM27762

Commit message: DRC pass
Check in before adding artwork and double checking parts.
Parts:
- added C13, C14: 2u2, Capacitor_SMD:C_0603_1608Metric, symbol vickys_symbols:GENERIC_C
- added LD6: APHHS1005LSECK/J3-PF, LED_SMD:LED_0402_1005Metric_Pad0.77x0.64mm_HandSolder, symbol vickys_symbols:APHHS1005LSECK/J3-PF
- C6, C7: footprint Capacitor_SMD:C_0805_2012Metric -> Capacitor_SMD:C_0603_1608Metric; Voltage Rating (none) -> 10V
- C8: footprint Capacitor_SMD:C_0603_1608Metric -> Capacitor_SMD:C_0402_1005Metric; Voltage Rating (none) -> 10V
- R17, R18, R20: footprint (none) -> Resistor_SMD:R_0402_1005Metric
- R19: value ~ -> 82K; footprint (none) -> Resistor_SMD:R_0402_1005Metric
- U3: footprint Package_SON:WSON-12-1EP_3x2mm_P0.5mm_EP1x2.65_ThermalVias -> Package_SON:WSON-12-1EP_3x2mm_P0.5mm_EP1x2.65
Connections:
- net +5V: now also C13.1, C14.1
- net GND: now also C13.2, C14.2
- net at R16.2: now also LD6.2 (A); no longer U3.1 (PGOOD)
- new net PGOOD: LD6.1 (K), U3.1 (PGOOD)
Other:
- title: (none) -> POWER

Commit message: A1 RELEASE
A1 released - pending feedback from PCBWay
Parts:
- C13, C14: Dielectric X7R -> X5R; MPN (none) -> GRM188Z71C225KE43D; Manufacturer (none) -> Murata; Mounting Type (none) -> SMT; Package/Case (none) -> 0603; RoHS (none) -> Y
- C6, C7: Dielectric X7R -> X5R; MPN (none) -> GRM188Z71C225KE43D; Manufacturer (none) -> Murata; Mounting Type (none) -> SMT; Package/Case (none) -> 0603; RoHS (none) -> Y; Voltage Rating 10V -> 16V
- C8: Dielectric X7R -> X5R; MPN (none) -> GRM155R61C105KA12D; Manufacturer (none) -> Murata; Mounting Type (none) -> SMT; Package/Case (none) -> 0402; RoHS (none) -> Y; Voltage Rating 10V -> 16V
- C9: Dielectric X7R -> X5R; MPN (none) -> GRM188R61C106MAALD; Manufacturer (none) -> Murata; Mounting Type (none) -> SMT; Package/Case (none) -> 0603; RoHS (none) -> Y; Voltage Rating 10V -> 16V
- R16: MPN (none) -> RC0603FR-0710KL; Manufacturer (none) -> YAGEO; Power Rating (none) -> 1/10W; RoHS (none) -> Y; Tolerance (none) -> 1%
- R17, R20: MPN (none) -> RC0402FR-0791KL; Manufacturer (none) -> YAGEO; Package/Case (none) -> 0402; Power Rating (none) -> 1/16W; RoHS (none) -> Y; Tolerance (none) -> 1%
- R18, R19: MPN (none) -> RC0402FR-0782KL; Manufacturer (none) -> YAGEO; Package/Case (none) -> 0402; Power Rating (none) -> 1/16W; RoHS (none) -> Y; Tolerance (none) -> 1%
- U3: MPN (none) -> LM27762DSS; Manufacturer (none) -> Texas Instruments; Mounting Type (none) -> SMT; Package/Case (none) -> 12-WSON; RoHS (none) -> Y
