File: vccs/sense_resistors.kicad_sch (KiCad schematic)
At the start: 15 parts, among them Q3 SIRA26DP, Q4 SIRA26DP, Q5 Si2318CDS, Q6 Si2318CDS, Q7 Si2318CDS

Commit message: DRC pass
Check in before adding artwork and double checking parts.
Parts:
- added LD1, LD2, LD3, LD4, LD5: APHHS1005LSECK/J3-PF, LED_SMD:LED_0402_1005Metric_Pad0.77x0.64mm_HandSolder, symbol vickys_symbols:APHHS1005LSECK/J3-PF
Connections:
- net GND: now also LD1.1 (K), LD2.1 (K), LD3.1 (K), LD4.1 (K), LD5.1 (K); no longer R11.2, R12.2, R13.2, R14.2, R15.2
- new net: LD4.2 (A), R14.2
- new net: LD5.2 (A), R15.2
- new net: LD2.2 (A), R12.2
- new net: LD3.2 (A), R13.2
- new net: LD1.2 (A), R11.2
Other:
- title: (none) -> SINK SENSE AND SELECT

Commit message: A1 RELEASE
A1 released - pending feedback from PCBWay
Parts:
- R10: MPN (none) -> RC1206FR-071KL; Manufacturer (none) -> YAGEO; Power Rating (none) -> 1/4W; RoHS (none) -> Y; Tolerance (none) -> 1%
- R11, R12, R13, R14, R15: MPN (none) -> RC0603FR-0710KL; Manufacturer (none) -> YAGEO; Power Rating (none) -> 1/10W; RoHS (none) -> Y; Tolerance (none) -> 1%
- R6: MPN (none) -> RL1206FR-070R33L; Manufacturer (none) -> YAGEO; Power Rating (none) -> 1/4W; RoHS (none) -> Y; Tolerance (none) -> 1%
- R7: MPN (none) -> RC1206FR-131RL; Manufacturer (none) -> YAGEO; Power Rating (none) -> 1/4W; RoHS (none) -> Y; Tolerance (none) -> 1%
- R8: MPN (none) -> RC1206FR-0710RL; Manufacturer (none) -> YAGEO; Power Rating (none) -> 1/4W; RoHS (none) -> Y; Tolerance (none) -> 1%
- R9: MPN (none) -> RC1206FR-07100RL; Manufacturer (none) -> YAGEO; Power Rating (none) -> 1/4W; RoHS (none) -> Y; Tolerance (none) -> 1%
Changed lines of the file:
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@@
 			)
 		)
-		(property "Manufacturer" ""
+		(property "Manufacturer" "YAGEO"
 			(at 115.57 128.27 0)
 			(effects
@@
 			)
 		)
-		(property "MPN" ""
+		(property "MPN" "RC0603FR-0710KL"
 			(at 115.57 128.27 0)
 			(effects
@@
 			)
 		)
-		(property "RoHS" ""
+		(property "RoHS" "Y"
 			(at 115.57 128.27 0)
 			(effects
@@
 			)
 		)
-		(property "Tolerance" ""
+		(property "Tolerance" "1%"
 			(at 115.57 128.27 0)
 			(effects
@@
 			)
 		)
-		(property "Power Rating" ""
+		(property "Power Rating" "1/10W"
 			(at 115.57 128.27 0)
 			(effects
@@
 			)
 		)
-		(property "Manufacturer" ""
+		(property "Manufacturer" "YAGEO"
 			(at 124.46 128.27 0)
 			(effects
@@
 			)
 		)
-		(property "MPN" ""
+		(property "MPN" "RC0603FR-0710KL"
 			(at 124.46 128.27 0)
 			(effects
@@
 			)
 		)
-		(property "RoHS" ""
+		(property "RoHS" "Y"
 			(at 124.46 128.27 0)
 			(effects
@@
 			)
 		)
-		(property "Tolerance" ""
+		(property "Tolerance" "1%"
 			(at 124.46 128.27 0)
 			(effects
@@
 			)
 		)
-		(property "Power Rating" ""
+		(property "Power Rating" "1/10W"
 			(at 124.46 128.27 0)
 			(effects
@@
 			)
 		)
-		(property "Manufacturer" ""
+		(property "Manufacturer" "YAGEO"
 			(at 193.04 128.27 0)
 			(effects
@@
 			)
 		)
-		(property "MPN" ""
+		(property "MPN" "RC1206FR-07100RL"
 			(at 193.04 128.27 0)
 			(effects
@@
 			)
 		)
-		(property "RoHS" ""
+		(property "RoHS" "Y"
 			(at 193.04 128.27 0)
 			(effects
@@
 			)
 		)
-		(property "Tolerance" ""
+		(property "Tolerance" "1%"
 			(at 193.04 128.27 0)
 			(effects
@@
 			)
 		)
-		(property "Power Rating" ""
+		(property "Power Rating" "1/4W"
 			(at 193.04 128.27 0)
 			(effects
@@
 			)
 		)
-		(property "Manufacturer" ""
+		(property "Manufacturer" "YAGEO"
 			(at 97.79 128.27 0)
 			(effects
@@
 			)
 		)
-		(property "MPN" ""
+		(property "MPN" "RC0603FR-0710KL"
 			(at 97.79 128.27 0)
 			(effects
@@
 			)
 		)
-		(property "RoHS" ""
+		(property "RoHS" "Y"
 			(at 97.79 128.27 0)
 			(effects
@@
 			)
 		)
-		(property "Tolerance" ""
+		(property "Tolerance" "1%"
 			(at 97.79 128.27 0)
 			(effects
@@
 			)
 		)
-		(property "Power Rating" ""
+		(property "Power Rating" "1/10W"
 			(at 97.79 128.27 0)
 			(effects
@@
 			)
 		)
-		(property "Manufacturer" ""
+		(property "Manufacturer" "YAGEO"
 			(at 106.68 128.27 0)
 			(effects
@@
 			)
 		)
-		(property "MPN" ""
+		(property "MPN" "RC0603FR-0710KL"
 			(at 106.68 128.27 0)
 			(effects
@@
 			)
 		)
-		(property "RoHS" ""
+		(property "RoHS" "Y"
 			(at 106.68 128.27 0)
 			(effects
@@
 			)
 		)
-		(property "Tolerance" ""
+		(property "Tolerance" "1%"
 			(at 106.68 128.27 0)
 			(effects
@@
 			)
 		)
-		(property "Power Rating" ""
+		(property "Power Rating" "1/10W"
 			(at 106.68 128.27 0)
 			(effects
@@
 			)
 		)
-		(property "Manufacturer" ""
+		(property "Manufacturer" "YAGEO"
 			(at 208.28 128.27 0)
 			(effects
@@
 			)
 		)
-		(property "MPN" ""
+		(property "MPN" "RC1206FR-071KL"
 			(at 208.28 128.27 0)
 			(effects
@@
 			)
 		)
-		(property "RoHS" ""
+		(property "RoHS" "Y"
 			(at 208.28 128.27 0)
 			(effects
@@
 			)
 		)
-		(property "Tolerance" ""
+		(property "Tolerance" "1%"
 			(at 208.28 128.27 0)
 			(effects
@@
 			)
 		)
-		(property "Power Rating" ""
+		(property "Power Rating" "1/4W"
 			(at 208.28 128.27 0)
 			(effects
@@
 			)
 		)
-		(property "Manufacturer" ""
+		(property "Manufacturer" "YAGEO"
 			(at 143.51 128.27 0)
 			(effects
@@
 			)
 		)
-		(property "MPN" ""
+		(property "MPN" "RL1206FR-070R33L"
 			(at 143.51 128.27 0)
 			(effects
@@
 			)
 		)
-		(property "RoHS" ""
+		(property "RoHS" "Y"
 			(at 143.51 128.27 0)
 			(effects
@@
 			)
 		)
-		(property "Tolerance" ""
+		(property "Tolerance" "1%"
 			(at 143.51 128.27 0)
 			(effects
@@
 			)
 		)
-		(property "Power Rating" ""
+		(property "Power Rating" "1/4W"
 			(at 143.51 128.27 0)
 			(effects
@@
 			)
 		)
-		(property "Manufacturer" ""
+		(property "Manufacturer" "YAGEO"
 			(at 161.29 128.27 0)
 			(effects
@@
 			)
 		)
-		(property "MPN" ""
+		(property "MPN" "RC1206FR-131RL"
 			(at 161.29 128.27 0)
 			(effects
@@
 			)
 		)
-		(property "RoHS" ""
+		(property "RoHS" "Y"
 			(at 161.29 128.27 0)
 			(effects
@@
 			)
 		)
-		(property "Tolerance" ""
+		(property "Tolerance" "1%"
 			(at 161.29 128.27 0)
 			(effects
@@
 			)
 		)
-		(property "Power Rating" ""
+		(property "Power Rating" "1/4W"
 			(at 161.29 128.27 0)
 			(effects
@@
 			)
 		)
-		(property "Manufacturer" ""
+		(property "Manufacturer" "YAGEO"
 			(at 177.8 128.27 0)
 			(effects
@@
 			)
 		)
-		(property "MPN" ""
+		(property "MPN" "RC1206FR-0710RL"
 			(at 177.8 128.27 0)
 			(effects
@@
 			)
 		)
-		(property "RoHS" ""
+		(property "RoHS" "Y"
 			(at 177.8 128.27 0)
 			(effects
@@
 			)
 		)
-		(property "Tolerance" ""
+		(property "Tolerance" "1%"
 			(at 177.8 128.27 0)
 			(effects
@@
 			)
 		)
-		(property "Power Rating" ""
+		(property "Power Rating" "1/4W"
 			(at 177.8 128.27 0)
 			(effects
@@
 			)
 		)
-		(property "Manufacturer" ""
+		(property "Manufacturer" "YAGEO"
 			(at 88.9 128.27 0)
 			(effects
@@
 			)
 		)
-		(property "MPN" ""
+		(property "MPN" "RC0603FR-0710KL"
 			(at 88.9 128.27 0)
 			(effects
@@
 			)
 		)
-		(property "RoHS" ""
+		(property "RoHS" "Y"
 			(at 88.9 128.27 0)
 			(effects
@@
 			)
 		)
-		(property "Tolerance" ""
+		(property "Tolerance" "1%"
 			(at 88.9 128.27 0)
 			(effects
@@
 			)
 		)
-		(property "Power Rating" ""
+		(property "Power Rating" "1/10W"
 			(at 88.9 128.27 0)
 			(effects
