File: vccs/sink.kicad_sch (KiCad schematic)
At the start: 16 parts, among them Q1 2SCR583D3, Q2 2SCR512P5, U1 TLV9002IDGK, U2 TLV9002IDGK

Commit message: DRC pass
Check in before adding artwork and double checking parts.
Parts:
- removed HS1: Heatsink_Pad, Heatsink:Heatsink_Fischer_FK24413D2PAK_26x13mm, symbol Mechanical:Heatsink_Pad
- added HS1: FK 244 13 D2 PAK, vickys_footprints:FK 244 13 D2 PAK, symbol vickys_symbols:FK 244 13 D2 PAK
- renumbered U2 to U1
Connections:
- net SINK_IN: now also HS1.1
- net at C1.2, R1.2: now also Q2.1 (B); no longer Q2.B
- net at R2.1: now also Q2.2 (C); no longer Q2.C
- net at Q1.1 (B): now also Q2.3 (E); no longer Q2.E
- net sense_resistors/IN renamed ISENSE
Other:
- title: (none) -> SINK

Commit message: A1 RELEASE
A1 released - pending feedback from PCBWay
Parts:
- C1: Dielectric (none) -> C0G/NP0; MPN (none) -> GRM1885C1H102JA01D; Manufacturer (none) -> Murata; RoHS (none) -> Y; Voltage Rating (none) -> 50V
- C2, C3: Dielectric (none) -> C0G/NP0; MPN (none) -> GRM1885C1H222JA01D; Manufacturer (none) -> Murata; RoHS (none) -> Y; Voltage Rating (none) -> 50V
- C4, C5: Dielectric (none) -> X7R; MPN (none) -> GCJ188R71H104KA12D; Manufacturer (none) -> Murata; RoHS (none) -> Y; Voltage Rating (none) -> 50V
- R1: MPN (none) -> RC0603FR-07100RL; Manufacturer (none) -> YAGEO; Power Rating (none) -> 1/10W; RoHS (none) -> Y
- R2: MPN (none) -> RC0603FR-0710RL; Manufacturer (none) -> YAGEO; Power Rating (none) -> 1/10W; RoHS (none) -> Y
- R21: value 10k -> 10K; MPN (none) -> RC0603FR-0710KL; Manufacturer (none) -> YAGEO; Power Rating (none) -> 1/10W; RoHS (none) -> Y
- R3, R4, R5: MPN (none) -> RC0603FR-071KL; Manufacturer (none) -> YAGEO; Power Rating (none) -> 1/10W; RoHS (none) -> Y
Changed lines of the file:
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@@
 			)
 		)
-		(property "Manufacturer" ""
+		(property "Manufacturer" "YAGEO"
 			(at 93.98 63.5 0)
 			(effects
@@
 			)
 		)
-		(property "MPN" ""
+		(property "MPN" "RC0603FR-071KL"
 			(at 93.98 63.5 0)
 			(effects
@@
 			)
 		)
-		(property "RoHS" ""
+		(property "RoHS" "Y"
 			(at 93.98 63.5 0)
 			(effects
@@
 			)
 		)
-		(property "Power Rating" ""
+		(property "Power Rating" "1/10W"
 			(at 93.98 63.5 0)
 			(effects
@@
 			)
 		)
-		(property "Manufacturer" ""
+		(property "Manufacturer" "YAGEO"
 			(at 147.32 66.04 0)
 			(effects
@@
 			)
 		)
-		(property "MPN" ""
+		(property "MPN" "RC0603FR-07100RL"
 			(at 147.32 66.04 0)
 			(effects
@@
 			)
 		)
-		(property "RoHS" ""
+		(property "RoHS" "Y"
 			(at 147.32 66.04 0)
 			(effects
@@
 			)
 		)
-		(property "Power Rating" ""
+		(property "Power Rating" "1/10W"
 			(at 147.32 66.04 0)
 			(effects
@@
 			)
 		)
-		(property "Manufacturer" ""
+		(property "Manufacturer" "Murata"
 			(at 31.75 172.72 0)
 			(effects
@@
 			)
 		)
-		(property "MPN" ""
+		(property "MPN" "GCJ188R71H104KA12D"
 			(at 31.75 172.72 0)
 			(effects
@@
 			)
 		)
-		(property "RoHS" ""
+		(property "RoHS" "Y"
 			(at 31.75 172.72 0)
 			(effects
@@
 			)
 		)
-		(property "Voltage Rating" ""
+		(property "Voltage Rating" "50V"
 			(at 31.75 172.72 0)
 			(effects
@@
 			)
 		)
-		(property "Dielectric" ""
+		(property "Dielectric" "X7R"
 			(at 31.75 172.72 0)
 			(effects
@@
 			)
 		)
-		(property "Value" "10k"
+		(property "Value" "10K"
 			(at 69.85 72.3899 0)
 			(effects
@@
 			)
 		)
-		(property "Manufacturer" ""
+		(property "Manufacturer" "YAGEO"
 			(at 67.31 71.12 0)
 			(effects
@@
 			)
 		)
-		(property "MPN" ""
+		(property "MPN" "RC0603FR-0710KL"
 			(at 67.31 71.12 0)
 			(effects
@@
 			)
 		)
-		(property "RoHS" ""
+		(property "RoHS" "Y"
 			(at 67.31 71.12 0)
 			(effects
@@
 			)
 		)
-		(property "Power Rating" ""
+		(property "Power Rating" "1/10W"
 			(at 67.31 71.12 0)
 			(effects
@@
 			)
 		)
-		(property "Manufacturer" ""
+		(property "Manufacturer" "Murata"
 			(at 133.35 82.55 0)
 			(effects
@@
 			)
 		)
-		(property "MPN" ""
+		(property "MPN" "GRM1885C1H222JA01D"
 			(at 133.35 82.55 0)
 			(effects
@@
 			)
 		)
-		(property "RoHS" ""
+		(property "RoHS" "Y"
 			(at 133.35 82.55 0)
 			(effects
@@
 			)
 		)
-		(property "Voltage Rating" ""
+		(property "Voltage Rating" "50V"
 			(at 133.35 82.55 0)
 			(effects
@@
 			)
 		)
-		(property "Dielectric" ""
+		(property "Dielectric" "C0G/NP0"
 			(at 133.35 82.55 0)
 			(effects
@@
 			)
 		)
-		(property "Manufacturer" ""
+		(property "Manufacturer" "Murata"
 			(at 147.32 54.61 0)
 			(effects
@@
 			)
 		)
-		(property "MPN" ""
+		(property "MPN" "GRM1885C1H102JA01D"
 			(at 147.32 54.61 0)
 			(effects
@@
 			)
 		)
-		(property "RoHS" ""
+		(property "RoHS" "Y"
 			(at 147.32 54.61 0)
 			(effects
@@
 			)
 		)
-		(property "Voltage Rating" ""
+		(property "Voltage Rating" "50V"
 			(at 147.32 54.61 0)
 			(effects
@@
 			)
 		)
-		(property "Dielectric" ""
+		(property "Dielectric" "C0G/NP0"
 			(at 147.32 54.61 0)
 			(effects
@@
 			)
 		)
-		(property "Manufacturer" ""
+		(property "Manufacturer" "YAGEO"
 			(at 140.97 99.06 0)
 			(effects
@@
 			)
 		)
-		(property "MPN" ""
+		(property "MPN" "RC0603FR-071KL"
 			(at 140.97 99.06 0)
 			(effects
@@
 			)
 		)
-		(property "RoHS" ""
+		(property "RoHS" "Y"
 			(at 140.97 99.06 0)
 			(effects
@@
 			)
 		)
-		(property "Power Rating" ""
+		(property "Power Rating" "1/10W"
 			(at 140.97 99.06 0)
 			(effects
@@
 			)
 		)
-		(property "Manufacturer" ""
+		(property "Manufacturer" "Murata"
 			(at 31.75 162.56 0)
 			(effects
@@
 			)
 		)
-		(property "MPN" ""
+		(property "MPN" "GCJ188R71H104KA12D"
 			(at 31.75 162.56 0)
 			(effects
@@
 			)
 		)
-		(property "RoHS" ""
+		(property "RoHS" "Y"
 			(at 31.75 162.56 0)
 			(effects
@@
 			)
 		)
-		(property "Voltage Rating" ""
+		(property "Voltage Rating" "50V"
 			(at 31.75 162.56 0)
 			(effects
@@
 			)
 		)
-		(property "Dielectric" ""
+		(property "Dielectric" "X7R"
 			(at 31.75 162.56 0)
 			(effects
@@
 			)
 		)
-		(property "Manufacturer" ""
+		(property "Manufacturer" "YAGEO"
 			(at 171.45 54.61 0)
 			(effects
@@
 			)
 		)
-		(property "MPN" ""
+		(property "MPN" "RC0603FR-0710RL"
 			(at 171.45 54.61 0)
 			(effects
@@
 			)
 		)
-		(property "RoHS" ""
+		(property "RoHS" "Y"
 			(at 171.45 54.61 0)
 			(effects
@@
 			)
 		)
-		(property "Power Rating" ""
+		(property "Power Rating" "1/10W"
 			(at 171.45 54.61 0)
 			(effects
@@
 			)
 		)
-		(property "Manufacturer" ""
+		(property "Manufacturer" "YAGEO"
 			(at 76.2 63.5 0)
 			(effects
@@
 			)
 		)
-		(property "MPN" ""
+		(property "MPN" "RC0603FR-071KL"
 			(at 76.2 63.5 0)
 			(effects
@@
 			)
 		)
-		(property "RoHS" ""
+		(property "RoHS" "Y"
 			(at 76.2 63.5 0)
 			(effects
@@
 			)
 		)
-		(property "Power Rating" ""
+		(property "Power Rating" "1/10W"
 			(at 76.2 63.5 0)
 			(effects
@@
 			)
 		)
-		(property "Manufacturer" ""
+		(property "Manufacturer" "Murata"
 			(at 85.09 69.85 0)
 			(effects
@@
 			)
 		)
-		(property "MPN" ""
+		(property "MPN" "GRM1885C1H222JA01D"
 			(at 85.09 69.85 0)
 			(effects
@@
 			)
 		)
-		(property "RoHS" ""
+		(property "RoHS" "Y"
 			(at 85.09 69.85 0)
 			(effects
@@
 			)
 		)
-		(property "Voltage Rating" ""
+		(property "Voltage Rating" "50V"
 			(at 85.09 69.85 0)
 			(effects
@@
 			)
 		)
-		(property "Dielectric" ""
+		(property "Dielectric" "C0G/NP0"
 			(at 85.09 69.85 0)
 			(effects
