File: vccs/vccs.kicad_pcb (KiCad board)
At the start: 4 copper layers, 78 x 50 mm, 67 parts, among them J1 575-4, J2 575-4, J3 B2B-PH-K, J4 3-1478978-1, J5 Conn_01x02_Socket, J6 Conn_01x10_Pin, J7 Conn_01x02_Pin, Q1 2SCR583D3, Q2 2SCR512P5, Q3 SIRA26DP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

Commit message: A1 RELEASE
A1 released - pending feedback from PCBWay
Changed lines of the file:
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@@
 		(tenting front back)
 		(pcbplotparams
-			(layerselection 0x00000000_00000000_55555555_5755f5ff)
+			(layerselection 0x00000000_00000000_55555555_5755f55f)
 			(plot_on_all_layers_selection 0x00000000_00000000_00000000_00000000)
 			(disableapertmacros no)
@@
 			(outputformat 1)
 			(mirror no)
-			(drillshape 1)
+			(drillshape 0)
 			(scaleselection 1)
-			(outputdirectory "")
+			(outputdirectory "project_outputs/")
 		)
 	)
@@
 		)
 	)
-	(gr_curve
-		(pts
-			(xy 123.4 56.6) (xy 122.7 60.3) (xy 120 59.7) (xy 120.3 58.4)
-		)
-		(stroke
-			(width 0.15)
-			(type solid)
-		)
-		(layer "F.SilkS")
-	)
 	(gr_line
