File: vccs/vccs.kicad_sch (KiCad schematic)
At the start: 0 parts

Commit message: Iterated sim and now putting into KiCad
Parts:
- added SW1: SW_DIP_x05, Button_Switch_SMD:SW_DIP_SPSTx06_Slide_9.78x17.42mm_W8.61mm_P2.54mm, symbol Switch:SW_DIP_x05
Connections:
- new net +5V: SW1.10, SW1.6, SW1.7, SW1.8, SW1.9
- new net SINK_SELECT0: SW1.1
- new net SINK_SELECT1: SW1.2
- new net SINK_SELECT2: SW1.3
- new net SINK_SELECT3: SW1.4
- new net SINK_SELECT4: SW1.5
Other:
- added sheet power (power.kicad_sch)
- added sheet sink (sink.kicad_sch)

Commit message: DRC pass
Check in before adding artwork and double checking parts.
Parts:
- removed SW1: SW_DIP_x05, Button_Switch_SMD:SW_DIP_SPSTx06_Slide_9.78x17.42mm_W8.61mm_P2.54mm, symbol Switch:SW_DIP_x05
- added C10, C11: 22u, Capacitor_SMD:C_1210_3225Metric_Pad1.33x2.70mm_HandSolder, symbol vickys_symbols:GENERIC_C
- added C12: 10u, Capacitor_SMD:C_0805_2012Metric, symbol vickys_symbols:GENERIC_C
- added D1: MBR0530, Diode_SMD:D_SOD-123, symbol Diode:MBR0530
- added H1, H2, H3, H4: M3, MountingHole:MountingHole_3.2mm_M3_Pad_Via, symbol Mechanical:MountingHole_Pad
- added J1, J2: 575-4, vickys_footprints:575-4, symbol vickys_symbols:575-4
- added J3: B2B-PH-K, Connector_JST:JST_PH_B2B-PH-K_1x02_P2.00mm_Vertical, symbol vickys_symbols:B2B-PH-K
- added J4: 3-1478978-1, vickys_footprints:3-1478978-1, symbol vickys_symbols:3-1478978-1
- added J5: Conn_01x02_Socket, Connector_JST:JST_PH_S2B-PH-K_1x02_P2.00mm_Horizontal, symbol Connector:Conn_01x02_Socket
- added J6: Conn_01x10_Pin, Connector_PinHeader_2.54mm:PinHeader_1x10_P2.54mm_Horizontal, symbol Connector:Conn_01x10_Pin
- added J7: Conn_01x02_Pin, Connector_PinHeader_2.54mm:PinHeader_1x02_P2.54mm_Vertical, symbol Connector:Conn_01x02_Pin
- added Q8: Si2318CDS, Package_TO_SOT_SMD:SOT-23-3, symbol vickys_symbols:Si2318CDS
- added R22, R23: 10K, Resistor_SMD:R_0603_1608Metric, symbol vickys_symbols:GENERIC_R
- added SW1: A6S-5104-H, vickys_footprints:A6S-5104-H, symbol vickys_symbols:A6S-5104-H
Connections:
- net +5V: now also C10.1, C11.1, C12.1, D1.1 (K), J3.1 (Pin_1), J5.1 (Pin_1), J6.10 (Pin_10), R22.1, SW1.1, SW1.2, SW1.3, SW1.4, SW1.5
- net SINK_SELECT0: now also J6.3 (Pin_3), SW1.10
- net SINK_SELECT1: now also J6.4 (Pin_4), SW1.9
- net SINK_SELECT2: now also J6.5 (Pin_5), SW1.8
- net SINK_SELECT3: now also J6.6 (Pin_6), SW1.7
- net SINK_SELECT4: now also J6.7 (Pin_7), SW1.6
- net sink/SINK_IN: now also J1.1 (Pin_1)
- new net: D1.2 (A), J3.2 (Pin_2), Q8.3 (D)
- new net FAN_EN: J6.8 (Pin_8), Q8.1 (G), R22.2, R23.1
- new net GND: C10.2, C11.2, C12.2, J2.1 (Pin_1), J4.2 (Ext), J5.2 (Pin_2), J6.2 (Pin_2), J6.9 (Pin_9), J7.2 (Pin_2), Q8.2 (S), R23.2
- new net VCONTROL: J4.1 (In), J6.1 (Pin_1)
- new net sink/ISENSE: J7.1 (Pin_1)
- no-connect marks 0 -> 4
Other:
- sheet sink ports: added ISENSE; removed none
- note added: "-->"
- note added: "0 -> 1V"
- note added: "0 -> 1V HiZ"
- note added: "COOLING FAN"
- note added: "CURRENT READ OUTPUT"
- note added: "EXTERNAL CONTROL"
- note added: "MOUNTING HOLES"
- note added: "POWER INPUT"
- note added: "Rail to be sunk"
- note added: "SINK & MANUAL SINK CONTROL"
- note added: "SINK CONTROL INPUT"
- note added: "SINK INPUT"
- note added: "SINK SELECT"
- note added: "SINK_SELECT0: 0-3A SINK_SELECT1: 0-1A SINK_SELECT2: 0-100mA SINK_SELECT3: 0-10mA SINK_SELECT4: 0-1mA"
- title: (none) -> MAIN

Commit message: A1 RELEASE
A1 released - pending feedback from PCBWay
Parts:
- C12: MPN (none) -> GRM21BZ71C106KE15L; Manufacturer (none) -> Murata; Mounting Type (none) -> SMT; Package/Case (none) -> 0805; RoHS (none) -> Y
- D1: value MBR0530 -> MBR0530T1G; MPN (none) -> MBR0530T1G; Manufacturer (none) -> onsemi; Mounting Type (none) -> SMT; Package/Case (none) -> SOD-123; RoHS (none) -> Y
- J5: value Conn_01x02_Socket -> S2B-PH-K-S; MPN (none) -> S2B-PH-K-S; Manufacturer (none) -> JST; Mounting Type (none) -> THT; RoHS (none) -> Y
- J6: value Conn_01x10_Pin -> M20-9961045; MPN (none) -> M20-9961045; Manufacturer (none) -> Harwin; Mounting Type (none) -> THT; RoHS (none) -> Y
- J7: value Conn_01x02_Pin -> M20-9990246; MPN (none) -> M20-9990246; Manufacturer (none) -> Harwin; Mounting Type (none) -> SMT; RoHS (none) -> Y
- R22, R23: MPN (none) -> RC0603FR-0710KL; Manufacturer (none) -> YAGEO; Power Rating (none) -> 1/10W; RoHS (none) -> Y
Changed lines of the file:
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@@
 	(text "SINK & MANUAL SINK CONTROL"
 		(exclude_from_sim no)
-		(at 104.14 72.136 0)
+		(at 96.012 73.152 0)
 		(effects
 			(font
@@
 	(wire
 		(pts
-			(xy 265.43 27.94) (xy 269.24 27.94)
+			(xy 267.97 27.94) (xy 269.24 27.94)
 		)
 		(stroke
@@
 	(wire
 		(pts
-			(xy 265.43 27.94) (xy 265.43 33.02)
+			(xy 267.97 27.94) (xy 267.97 33.02)
 		)
 		(stroke
@@
 	(wire
 		(pts
-			(xy 265.43 33.02) (xy 251.46 33.02)
+			(xy 267.97 33.02) (xy 251.46 33.02)
 		)
 		(stroke
@@
 		(dnp no)
 		(property "Reference" "J7"
-			(at 234.315 106.68 0)
+			(at 233.934 106.68 0)
 			(effects
 				(font
@@
 			)
 		)
-		(property "Value" "Conn_01x02_Pin"
-			(at 234.315 109.22 0)
+		(property "Value" "M20-9990246"
+			(at 228.092 108.966 0)
 			(effects
 				(font
@@
 			)
 		)
+		(property "Manufacturer" "Harwin"
+			(at 234.95 111.76 0)
+			(effects
+				(font
+					(size 1.27 1.27)
+				)
+				(hide yes)
+			)
+		)
+		(property "MPN" "M20-9990246"
+			(at 234.95 111.76 0)
+			(effects
+				(font
+					(size 1.27 1.27)
+				)
+				(hide yes)
+			)
+		)
+		(property "Mounting Type" "SMT"
+			(at 234.95 111.76 0)
+			(effects
+				(font
+					(size 1.27 1.27)
+				)
+				(hide yes)
+			)
+		)
+		(property "RoHS" "Y"
+			(at 234.95 111.76 0)
+			(effects
+				(font
+					(size 1.27 1.27)
+				)
+				(hide yes)
+			)
+		)
 		(pin "2"
 		)
@@
 			)
 		)
-		(property "Manufacturer" ""
+		(property "Manufacturer" "Murata"
 			(at 50.8 36.83 0)
 			(effects
@@
 			)
 		)
-		(property "MPN" ""
+		(property "MPN" "GRM21BZ71C106KE15L"
 			(at 50.8 36.83 0)
 			(effects
@@
 			)
 		)
-		(property "Package/Case" ""
+		(property "Package/Case" "0805"
 			(at 50.8 53.34 0)
 			(effects
@@
 			)
 		)
-		(property "Mounting Type" ""
+		(property "Mounting Type" "SMT"
 			(at 50.8 55.88 0)
 			(effects
@@
 			)
 		)
-		(property "RoHS" ""
+		(property "RoHS" "Y"
 			(at 50.8 36.83 0)
 			(effects
@@
 			)
 		)
-		(property "Value" "MBR0530"
+		(property "Value" "MBR0530T1G"
 			(at 254 30.1624 90)
 			(effects
@@
 			)
 		)
-		(property "Datasheet" "http://www.mccsemi.com/up_pdf/MBR0520~MBR0580(SOD123).pdf"
+		(property "Datasheet" "https://www.onsemi.com/pdf/datasheet/mbr0530t1-d.pdf"
 			(at 251.46 29.21 0)
 			(effects
@@
 			)
 		)
+		(property "Manufacturer" "onsemi"
+			(at 251.46 29.21 90)
+			(effects
+				(font
+					(size 1.27 1.27)
+				)
+				(hide yes)
+			)
+		)
+		(property "MPN" "MBR0530T1G"
+			(at 251.46 29.21 90)
+			(effects
+				(font
+					(size 1.27 1.27)
+				)
+				(hide yes)
+			)
+		)
+		(property "Mounting Type" "SMT"
+			(at 251.46 29.21 90)
+			(effects
+				(font
+					(size 1.27 1.27)
+				)
+				(hide yes)
+			)
+		)
+		(property "Package/Case" "SOD-123"
+			(at 251.46 29.21 90)
+			(effects
+				(font
+					(size 1.27 1.27)
+				)
+				(hide yes)
+			)
+		)
+		(property "RoHS" "Y"
+			(at 251.46 29.21 90)
+			(effects
+				(font
+					(size 1.27 1.27)
+				)
+				(hide yes)
+			)
+		)
 		(pin "2"
 		)
@@
 			)
 		)
-		(property "Value" "Conn_01x10_Pin"
-			(at 171.45 34.798 0)
+		(property "Value" "M20-9961045"
+			(at 170.688 34.798 0)
 			(effects
 				(font
@@
 			)
 		)
+		(property "Manufacturer" "Harwin"
+			(at 161.29 35.56 0)
+			(effects
+				(font
+					(size 1.27 1.27)
+				)
+				(hide yes)
+			)
+		)
+		(property "MPN" "M20-9961045"
+			(at 161.29 35.56 0)
+			(effects
+				(font
+					(size 1.27 1.27)
+				)
+				(hide yes)
+			)
+		)
+		(property "Package/Case" ""
+			(at 161.29 35.56 0)
+			(effects
+				(font
+					(size 1.27 1.27)
+				)
+				(hide yes)
+			)
+		)
+		(property "Mounting Type" "THT"
+			(at 161.29 35.56 0)
+			(effects
+				(font
+					(size 1.27 1.27)
+				)
+				(hide yes)
+			)
+		)
+		(property "RoHS" "Y"
+			(at 161.29 35.56 0)
+			(effects
+				(font
+					(size 1.27 1.27)
+				)
+				(hide yes)
+			)
+		)
 		(pin "4"
 		)
@@
 		(dnp no)
 		(property "Reference" "J3"
-			(at 273.685 20.32 0)
+			(at 271.78 30.226 0)
 			(effects
 				(font
@@
 		)
 		(property "Value" "B2B-PH-K"
-			(at 273.685 22.86 0)
+			(at 276.098 32.766 0)
 			(effects
 				(font
@@
 			)
 		)
-		(property "Manufacturer" ""
+		(property "Manufacturer" "YAGEO"
 			(at 232.41 30.48 0)
 			(effects
@@
 			)
 		)
-		(property "MPN" ""
+		(property "MPN" "RC0603FR-0710KL"
 			(at 232.41 30.48 0)
 			(effects
@@
 			)
 		)
-		(property "RoHS" ""
+		(property "RoHS" "Y"
 			(at 232.41 30.48 0)
 			(effects
@@
 			)
 		)
-		(property "Power Rating" ""
+		(property "Power Rating" "1/10W"
 			(at 232.41 30.48 0)
 			(effects
@@
 			)
 		)
-		(property "Manufacturer" ""
+		(property "Manufacturer" "YAGEO"
 			(at 234.95 43.18 0)
 			(effects
@@
 			)
 		)
-		(property "MPN" ""
+		(property "MPN" "RC0603FR-0710KL"
 			(at 234.95 43.18 0)
 			(effects
@@
 			)
 		)
-		(property "RoHS" ""
+		(property "RoHS" "Y"
 			(at 234.95 43.18 0)
 			(effects
@@
 			)
 		)
-		(property "Power Rating" ""
+		(property "Power Rating" "1/10W"
 			(at 234.95 43.18 0)
 			(effects
@@
 			)
 		)
-		(property "Value" "Conn_01x02_Socket"
+		(property "Value" "S2B-PH-K-S"
 			(at 31.115 29.21 0)
 			(effects
@@
 			(at 30.48 31.75 0)
 			(effects
+				(font
+					(size 1.27 1.27)
+				)
+				(hide yes)
+			)
+		)
+		(property "Manufacturer" "JST"
+			(at 30.48 31.75 0)
+			(effects
+				(font
+					(size 1.27 1.27)
+				)
+				(hide yes)
+			)
+		)
+		(property "MPN" "S2B-PH-K-S"
+			(at 30.48 31.75 0)
+			(effects
+				(font
+					(size 1.27 1.27)
+				)
+				(hide yes)
+			)
+		)
+		(property "Mounting Type" "THT"
+			(at 30.48 31.75 0)
+			(effects
+				(font
+					(size 1.27 1.27)
+				)
+				(hide yes)
+			)
+		)
+		(property "RoHS" "Y"
+			(at 30.48 31.75 0)
+			(effects
